File: LM1117.kicad_sch (KiCad schematic)
At the start: 3 parts, among them U2 LM1117MP-3.3

Commit message: Update schematics, power flags and PCB design
Parts:
- renumbered C8 to C11, C9 to C12, U2 to U3
Changed lines of the file:
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@@
 		(dnp no)
 		(fields_autoplaced yes)
-		(property "Reference" "#PWR016"
+		(property "Reference" "#PWR025"
 			(at 54.61 43.18 0)
 			(hide yes)
@@
 			(project "stm32f103c8t6"
 				(path "/bd823326-686b-4669-b4e8-652a43eb6bb4/01d50728-be12-47d4-a3b3-3530cdf67424"
-					(reference "#PWR016")
+					(reference "#PWR025")
 					(unit 1)
 				)
@@
 		(dnp no)
 		(fields_autoplaced yes)
-		(property "Reference" "#PWR012"
+		(property "Reference" "#PWR026"
 			(at 54.61 80.01 0)
 			(hide yes)
@@
 			(project "stm32f103c8t6"
 				(path "/bd823326-686b-4669-b4e8-652a43eb6bb4/01d50728-be12-47d4-a3b3-3530cdf67424"
-					(reference "#PWR012")
+					(reference "#PWR026")
 					(unit 1)
 				)
@@
 		(dnp no)
 		(fields_autoplaced yes)
-		(property "Reference" "#PWR013"
+		(property "Reference" "#PWR029"
 			(at 104.14 80.01 0)
 			(hide yes)
@@
 			(project "stm32f103c8t6"
 				(path "/bd823326-686b-4669-b4e8-652a43eb6bb4/01d50728-be12-47d4-a3b3-3530cdf67424"
-					(reference "#PWR013")
+					(reference "#PWR029")
 					(unit 1)
 				)
@@
 		(dnp no)
 		(fields_autoplaced yes)
-		(property "Reference" "U2"
+		(property "Reference" "U3"
 			(at 80.01 43.18 0)
 			(show_name no)
@@
 			(project "stm32f103c8t6"
 				(path "/bd823326-686b-4669-b4e8-652a43eb6bb4/01d50728-be12-47d4-a3b3-3530cdf67424"
-					(reference "U2")
+					(reference "U3")
 					(unit 1)
 				)
@@
 		(dnp no)
 		(fields_autoplaced yes)
-		(property "Reference" "#PWR015"
+		(property "Reference" "#PWR028"
 			(at 104.14 43.18 0)
 			(hide yes)
@@
 			(project "stm32f103c8t6"
 				(path "/bd823326-686b-4669-b4e8-652a43eb6bb4/01d50728-be12-47d4-a3b3-3530cdf67424"
-					(reference "#PWR015")
+					(reference "#PWR028")
 					(unit 1)
 				)
@@
 		(dnp no)
 		(fields_autoplaced yes)
-		(property "Reference" "C8"
+		(property "Reference" "C11"
 			(at 58.42 60.9599 0)
 			(show_name no)
@@
 			(project "stm32f103c8t6"
 				(path "/bd823326-686b-4669-b4e8-652a43eb6bb4/01d50728-be12-47d4-a3b3-3530cdf67424"
-					(reference "C8")
+					(reference "C11")
 					(unit 1)
 				)
@@
 		(dnp no)
 		(fields_autoplaced yes)
-		(property "Reference" "C9"
+		(property "Reference" "C12"
 			(at 107.95 60.9599 0)
 			(show_name no)
@@
 			(project "stm32f103c8t6"
 				(path "/bd823326-686b-4669-b4e8-652a43eb6bb4/01d50728-be12-47d4-a3b3-3530cdf67424"
-					(reference "C9")
+					(reference "C12")
 					(unit 1)
 				)
@@
 		(dnp no)
 		(fields_autoplaced yes)
-		(property "Reference" "#PWR014"
+		(property "Reference" "#PWR027"
 			(at 80.01 71.12 0)
 			(hide yes)
@@
 			(project "stm32f103c8t6"
 				(path "/bd823326-686b-4669-b4e8-652a43eb6bb4/01d50728-be12-47d4-a3b3-3530cdf67424"
-					(reference "#PWR014")
-					(unit 1)
-				)
+					(reference "#PWR027")
+					(unit 1)
+				)
