File: STM32F103C8_MCU.kicad_sch (KiCad schematic)
At the start: 12 parts, among them J1 Header Socket 1X5, SW1 SW_SPST, U1 STM32F103C8T6, Y1 Crystal

Commit message: Update USB-C and FTDI circuits and add button and potentiometer sheets
Parts:
- added C10, C11: 20pF(1608), symbol Device:C
- added R19, R20: 22R(1608), symbol Device:R_US
- added R27, R28: 10KR(1608), symbol Device:R_US
- added R6: 0R(1608), symbol Device:R_US
- Y1: value Crystal -> 8MHz
Connections:
- net +3V3: now also R27.1, R28.1
- net GND: now also C10.1, C11.2
- net OSC_IN: now also C11.1
- net OSC_OUT: now also C10.2, R6.2; no longer U1.6 (OSC_OUT)
- net ADC_IN0: now reaches U1.10 (PA0-WKUP)
- net ADC_IN1: now reaches U1.11 (PA1)
- net ADC_IN2: now reaches U1.12 (PA2)
- net ADC_IN3: now reaches U1.13 (PA3)
- net IO_IN_SW1: now reaches U1.14 (PA4)
- net IO_IN_SW2: now reaches U1.15 (PA5)
- net IO_IN_SW3: now reaches U1.16 (PA6)
- net IO_IN_SW4: now reaches U1.17 (PA7)
- net TIM2_CH1_PWM: now reaches U1.38 (PA15)
- net at U1.42 (PB6): now also R19.1
- net at U1.43 (PB7): now also R20.1
- new net: R6.1, U1.6 (OSC_OUT)
- new net MCU_UART1_RX: R20.2, R28.2
- new net MCU_UART1_TX: R19.2, R27.2
Other:
- moved on the sheet: J1, Y1

Commit message: Update schematics, power flags and PCB design
Parts:
- added R12, R13: 22R(1608), Resistor_SMD:R_0603_1608Metric, symbol Device:R_US
- C2: renamed from C10; footprint (none) -> Capacitor_SMD:C_0603_1608Metric
- C3: renamed from C11; footprint (none) -> Capacitor_SMD:C_0603_1608Metric
- J3: renamed from J1; footprint (none) -> Connector_PinHeader_2.54mm:PinHeader_1x05_P2.54mm_Vertical
- R10: renamed from R19; footprint (none) -> Resistor_SMD:R_0603_1608Metric
- R11: renamed from R20; footprint (none) -> Resistor_SMD:R_0603_1608Metric
- R14: renamed from R6; footprint (none) -> Resistor_SMD:R_0603_1608Metric
- R15: renamed from R1; footprint (none) -> Resistor_SMD:R_0603_1608Metric
- R8: renamed from R27; footprint (none) -> Resistor_SMD:R_0603_1608Metric
- R9: renamed from R28; footprint (none) -> Resistor_SMD:R_0603_1608Metric
- SW1: footprint (none) -> Button_Switch_THT:SW_PUSH_6mm_H5mm
- U2: renamed from U1; footprint LQFP48_STM -> jwj_lib:LQFP48_STM
- Y1: footprint (none) -> Crystal:Crystal_SMD_HC49-SD
- renumbered C4 to C10, C7 to C4, C1 to C5, C5 to C6, C2 to C7, C6 to C8, C3 to C9
Connections:
- net at U2.21 (PB10): now also R12.1
- net at U2.22 (PB11): now also R13.1
- new net MCU_UART3_RX: R13.2
- new net MCU_UART3_TX: R12.2
- no-connect marks 0 -> 16
