File: button.kicad_sch (KiCad schematic)
At the start: 12 parts, among them SW2 SW_SPST, SW3 SW_SPST, SW4 SW_SPST, SW5 SW_SPST

Commit message: Update schematics, power flags and PCB design
Parts:
- R20: renamed from R7; footprint (none) -> Resistor_SMD:R_0603_1608Metric
- R21: renamed from R8; footprint (none) -> Resistor_SMD:R_0603_1608Metric
- R22: renamed from R9; footprint (none) -> Resistor_SMD:R_0603_1608Metric
- R23: renamed from R10; footprint (none) -> Resistor_SMD:R_0603_1608Metric
- R24: renamed from R11; footprint (none) -> Resistor_SMD:R_0603_1608Metric
- R25: renamed from R12; footprint (none) -> Resistor_SMD:R_0603_1608Metric
- R26: renamed from R13; footprint (none) -> Resistor_SMD:R_0603_1608Metric
- R27: renamed from R14; footprint (none) -> Resistor_SMD:R_0603_1608Metric
- SW2, SW3, SW4, SW5: footprint (none) -> Button_Switch_THT:SW_PUSH_6mm_H5mm
Changed lines of the file:
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@@
 		(dnp no)
 		(fields_autoplaced yes)
-		(property "Reference" "#PWR021"
+		(property "Reference" "#PWR033"
 			(at 115.57 33.02 0)
 			(hide yes)
@@
 			(project "stm32f103c8t6"
 				(path "/bd823326-686b-4669-b4e8-652a43eb6bb4/5c56460d-9d96-44fe-8857-0395c646f3b3"
-					(reference "#PWR021")
+					(reference "#PWR033")
 					(unit 1)
 				)
@@
 		(in_pos_files yes)
 		(dnp no)
-		(property "Reference" "R10"
+		(property "Reference" "R23"
 			(at 134.62 55.88 90)
 			(show_name no)
@@
 			)
 		)
-		(property "Footprint" ""
+		(property "Footprint" "Resistor_SMD:R_0603_1608Metric"
 			(at 134.366 54.356 90)
 			(hide yes)
@@
 			(project "stm32f103c8t6"
 				(path "/bd823326-686b-4669-b4e8-652a43eb6bb4/5c56460d-9d96-44fe-8857-0395c646f3b3"
-					(reference "R10")
+					(reference "R23")
 					(unit 1)
 				)
@@
 		(dnp no)
 		(fields_autoplaced yes)
-		(property "Reference" "#PWR024"
+		(property "Reference" "#PWR036"
 			(at 167.64 87.63 0)
 			(hide yes)
@@
 			(project "stm32f103c8t6"
 				(path "/bd823326-686b-4669-b4e8-652a43eb6bb4/5c56460d-9d96-44fe-8857-0395c646f3b3"
-					(reference "#PWR024")
+					(reference "#PWR036")
 					(unit 1)
 				)
@@
 		(in_pos_files yes)
 		(dnp no)
-		(property "Reference" "R13"
+		(property "Reference" "R26"
 			(at 228.346 40.5702 0)
 			(show_name no)
@@
 			)
 		)
-		(property "Footprint" ""
+		(property "Footprint" "Resistor_SMD:R_0603_1608Metric"
 			(at 223.774 42.3482 90)
 			(hide yes)
@@
 			(project "stm32f103c8t6"
 				(path "/bd823326-686b-4669-b4e8-652a43eb6bb4/5c56460d-9d96-44fe-8857-0395c646f3b3"
-					(reference "R13")
+					(reference "R26")
 					(unit 1)
 				)
@@
 		(dnp no)
 		(fields_autoplaced yes)
-		(property "Reference" "#PWR020"
+		(property "Reference" "#PWR032"
 			(at 54.61 87.63 0)
 			(hide yes)
@@
 			(project "stm32f103c8t6"
 				(path "/bd823326-686b-4669-b4e8-652a43eb6bb4/5c56460d-9d96-44fe-8857-0395c646f3b3"
-					(reference "#PWR020")
+					(reference "#PWR032")
 					(unit 1)
 				)
@@
 		(dnp no)
 		(fields_autoplaced yes)
-		(property "Reference" "#PWR023"
+		(property "Reference" "#PWR035"
 			(at 167.64 33.02 0)
 			(hide yes)
@@
 			(project "stm32f103c8t6"
 				(path "/bd823326-686b-4669-b4e8-652a43eb6bb4/5c56460d-9d96-44fe-8857-0395c646f3b3"
-					(reference "#PWR023")
+					(reference "#PWR035")
 					(unit 1)
 				)
@@
 		(in_pos_files yes)
 		(dnp no)
-		(property "Reference" "R14"
+		(property "Reference" "R27"
 			(at 243.84 56.5722 90)
 			(show_name no)
@@
 			)
 		)
-		(property "Footprint" ""
+		(property "Footprint" "Resistor_SMD:R_0603_1608Metric"
 			(at 243.586 55.0482 90)
 			(hide yes)
@@
 			(project "stm32f103c8t6"
 				(path "/bd823326-686b-4669-b4e8-652a43eb6bb4/5c56460d-9d96-44fe-8857-0395c646f3b3"
-					(reference "R14")
+					(reference "R27")
 					(unit 1)
 				)
@@
 		(dnp no)
 		(fields_autoplaced yes)
-		(property "Reference" "#PWR022"
+		(property "Reference" "#PWR034"
 			(at 115.57 87.63 0)
 			(hide yes)
@@
 			(project "stm32f103c8t6"
 				(path "/bd823326-686b-4669-b4e8-652a43eb6bb4/5c56460d-9d96-44fe-8857-0395c646f3b3"
-					(reference "#PWR022")
+					(reference "#PWR034")
 					(unit 1)
 				)
@@
 			)
 		)
-		(property "Footprint" ""
+		(property "Footprint" "Button_Switch_THT:SW_PUSH_6mm_H5mm"
 			(at 115.57 67.31 0)
 			(hide yes)
@@
 		(in_pos_files yes)
 		(dnp no)
-		(property "Reference" "R7"
+		(property "Reference" "R20"
 			(at 58.166 39.878 0)
 			(show_name no)
@@
 			)
 		)
-		(property "Footprint" ""
+		(property "Footprint" "Resistor_SMD:R_0603_1608Metric"
 			(at 53.594 41.656 90)
 			(hide yes)
@@
 			(project "stm32f103c8t6"
 				(path "/bd823326-686b-4669-b4e8-652a43eb6bb4/5c56460d-9d96-44fe-8857-0395c646f3b3"
-					(reference "R7")
+					(reference "R20")
 					(unit 1)
 				)
@@
 		(dnp no)
 		(fields_autoplaced yes)
-		(property "Reference" "#PWR026"
+		(property "Reference" "#PWR038"
 			(at 224.79 88.3222 0)
 			(hide yes)
@@
 			(project "stm32f103c8t6"
 				(path "/bd823326-686b-4669-b4e8-652a43eb6bb4/5c56460d-9d96-44fe-8857-0395c646f3b3"
-					(reference "#PWR026")
+					(reference "#PWR038")
 					(unit 1)
 				)
@@
 		(in_pos_files yes)
 		(dnp no)
-		(property "Reference" "R11"
+		(property "Reference" "R24"
 			(at 171.196 39.878 0)
 			(show_name no)
@@
 			)
 		)
-		(property "Footprint" ""
+		(property "Footprint" "Resistor_SMD:R_0603_1608Metric"
 			(at 166.624 41.656 90)
 			(hide yes)
@@
 			(project "stm32f103c8t6"
 				(path "/bd823326-686b-4669-b4e8-652a43eb6bb4/5c56460d-9d96-44fe-8857-0395c646f3b3"
-					(reference "R11")
+					(reference "R24")
 					(unit 1)
 				)
@@
 		(in_pos_files yes)
 		(dnp no)
-		(property "Reference" "R8"
+		(property "Reference" "R21"
 			(at 73.66 55.88 90)
 			(show_name no)
@@
 			)
 		)
-		(property "Footprint" ""
+		(property "Footprint" "Resistor_SMD:R_0603_1608Metric"
 			(at 73.406 54.356 90)
 			(hide yes)
@@
 			(project "stm32f103c8t6"
 				(path "/bd823326-686b-4669-b4e8-652a43eb6bb4/5c56460d-9d96-44fe-8857-0395c646f3b3"
-					(reference "R8")
+					(reference "R21")
 					(unit 1)
 				)
@@
 			)
 		)
-		(property "Footprint" ""
+		(property "Footprint" "Button_Switch_THT:SW_PUSH_6mm_H5mm"
 			(at 224.79 68.0022 0)
 			(hide yes)
@@
 			)
 		)
-		(property "Footprint" ""
+		(property "Footprint" "Button_Switch_THT:SW_PUSH_6mm_H5mm"
 			(at 167.64 67.31 0)
 			(hide yes)
@@
 		(dnp no)
 		(fields_autoplaced yes)
-		(property "Reference" "#PWR025"
+		(property "Reference" "#PWR037"
 			(at 224.79 33.7122 0)
 			(hide yes)
@@
 			(project "stm32f103c8t6"
 				(path "/bd823326-686b-4669-b4e8-652a43eb6bb4/5c56460d-9d96-44fe-8857-0395c646f3b3"
-					(reference "#PWR025")
+					(reference "#PWR037")
 					(unit 1)
 				)
@@
 			)
 		)
-		(property "Footprint" ""
+		(property "Footprint" "Button_Switch_THT:SW_PUSH_6mm_H5mm"
 			(at 54.61 67.31 0)
 			(hide yes)
@@
 		(in_pos_files yes)
 		(dnp no)
-		(property "Reference" "R12"
+		(property "Reference" "R25"
 			(at 186.69 55.88 90)
 			(show_name no)
@@
 			)
 		)
-		(property "Footprint" ""
+		(property "Footprint" "Resistor_SMD:R_0603_1608Metric"
 			(at 186.436 54.356 90)
 			(hide yes)
@@
 			(project "stm32f103c8t6"
 				(path "/bd823326-686b-4669-b4e8-652a43eb6bb4/5c56460d-9d96-44fe-8857-0395c646f3b3"
-					(reference "R12")
+					(reference "R25")
 					(unit 1)
 				)
@@
 		(in_pos_files yes)
 		(dnp no)
-		(property "Reference" "R9"
+		(property "Reference" "R22"
 			(at 119.126 39.878 0)
 			(show_name no)
@@
 			)
 		)
-		(property "Footprint" ""
+		(property "Footprint" "Resistor_SMD:R_0603_1608Metric"
 			(at 114.554 41.656 90)
 			(hide yes)
@@
 			(project "stm32f103c8t6"
 				(path "/bd823326-686b-4669-b4e8-652a43eb6bb4/5c56460d-9d96-44fe-8857-0395c646f3b3"
-					(reference "R9")
+					(reference "R22")
 					(unit 1)
 				)
@@
 		(dnp no)
 		(fields_autoplaced yes)
-		(property "Reference" "#PWR019"
+		(property "Reference" "#PWR031"
 			(at 54.61 33.02 0)
 			(hide yes)
@@
 			(project "stm32f103c8t6"
 				(path "/bd823326-686b-4669-b4e8-652a43eb6bb4/5c56460d-9d96-44fe-8857-0395c646f3b3"
-					(reference "#PWR019")
-					(unit 1)
-				)
+					(reference "#PWR031")
+					(unit 1)
+				)
