File: ftdi.kicad_sch (KiCad schematic)
At the start: 10 parts, among them U3 FT232RL

Commit message: Update schematics, power flags and PCB design
Parts:
- D5, D6: footprint (none) -> LED_SMD:LED_0603_1608Metric
- R32: renamed from R21; footprint (none) -> Resistor_SMD:R_0603_1608Metric
- R33: renamed from R22; footprint (none) -> Resistor_SMD:R_0603_1608Metric
- R34: renamed from R23; footprint (none) -> Resistor_SMD:R_0603_1608Metric
- renumbered C16 to C17, C19 to C18, C17 to C19, C18 to C20, U3 to U4
Connections:
- net GND: now also U4.26 (TEST)
- no-connect marks 0 -> 11
Changed lines of the file:
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@@
 		(color 0 0 0 0)
 	)
+	(no_connect
+		(at 176.53 83.82)
+	)
+	(no_connect
+		(at 176.53 81.28)
+	)
+	(no_connect
+		(at 176.53 106.68)
+	)
+	(no_connect
+		(at 176.53 86.36)
+	)
+	(no_connect
+		(at 176.53 109.22)
+	)
+	(no_connect
+		(at 176.53 93.98)
+	)
+	(no_connect
+		(at 135.89 104.14)
+	)
+	(no_connect
+		(at 176.53 88.9)
+	)
+	(no_connect
+		(at 176.53 91.44)
+	)
+	(no_connect
+		(at 176.53 111.76)
+	)
+	(no_connect
+		(at 135.89 99.06)
+	)
 	(wire
 		(pts
@@
 	(wire
 		(pts
+			(xy 132.08 111.76) (xy 132.08 118.11)
+		)
+		(stroke
+			(width 0)
+			(type default)
+		)
+	)
+	(wire
+		(pts
 			(xy 161.29 121.92) (xy 158.75 121.92)
 		)
@@
 		(pts
 			(xy 209.55 101.6) (xy 218.44 101.6)
+		)
+		(stroke
+			(width 0)
+			(type default)
+		)
+	)
+	(wire
+		(pts
+			(xy 135.89 111.76) (xy 132.08 111.76)
 		)
 		(stroke
@@
 		(in_pos_files yes)
 		(dnp no)
-		(property "Reference" "#PWR036"
+		(property "Reference" "#PWR054"
 			(at 158.75 64.77 0)
 			(hide yes)
@@
 			(project "stm32f103c8t6"
 				(path "/bd823326-686b-4669-b4e8-652a43eb6bb4/b6e9bfc2-4cf7-4d7e-81c9-9912399d557a"
-					(reference "#PWR036")
+					(reference "#PWR054")
 					(unit 1)
 				)
@@
 		(in_pos_files yes)
 		(dnp no)
-		(property "Reference" "R22"
+		(property "Reference" "R33"
 			(at 205.74 97.536 90)
 			(show_name no)
@@
 			)
 		)
-		(property "Footprint" ""
+		(property "Footprint" "Resistor_SMD:R_0603_1608Metric"
 			(at 205.994 102.616 90)
 			(hide yes)
@@
 			(project "stm32f103c8t6"
 				(path "/bd823326-686b-4669-b4e8-652a43eb6bb4/b6e9bfc2-4cf7-4d7e-81c9-9912399d557a"
-					(reference "R22")
+					(reference "R33")
 					(unit 1)
 				)
@@
 		(dnp no)
 		(fields_autoplaced yes)
-		(property "Reference" "#PWR039"
+		(property "Reference" "#PWR051"
 			(at 151.13 130.81 0)
 			(hide yes)
@@
 			(project "stm32f103c8t6"
 				(path "/bd823326-686b-4669-b4e8-652a43eb6bb4/b6e9bfc2-4cf7-4d7e-81c9-9912399d557a"
-					(reference "#PWR039")
+					(reference "#PWR051")
 					(unit 1)
 				)
@@
 		(dnp no)
 		(fields_autoplaced yes)
-		(property "Reference" "#PWR040"
+		(property "Reference" "#PWR053"
 			(at 156.21 130.81 0)
 			(hide yes)
@@
 			(project "stm32f103c8t6"
 				(path "/bd823326-686b-4669-b4e8-652a43eb6bb4/b6e9bfc2-4cf7-4d7e-81c9-9912399d557a"
-					(reference "#PWR040")
+					(reference "#PWR053")
 					(unit 1)
 				)
@@
 		(dnp no)
 		(fields_autoplaced yes)
-		(property "Reference" "C19"
+		(property "Reference" "C18"
 			(at 121.92 68.58 90)
 			(show_name no)
@@
 			(project "stm32f103c8t6"
 				(path "/bd823326-686b-4669-b4e8-652a43eb6bb4/b6e9bfc2-4cf7-4d7e-81c9-9912399d557a"
-					(reference "C19")
+					(reference "C18")
 					(unit 1)
 				)
@@
 		(dnp no)
 		(fields_autoplaced yes)
-		(property "Reference" "#PWR037"
+		(property "Reference" "#PWR050"
 			(at 114.3 66.04 0)
 			(hide yes)
@@
 			(project "stm32f103c8t6"
 				(path "/bd823326-686b-4669-b4e8-652a43eb6bb4/b6e9bfc2-4cf7-4d7e-81c9-9912399d557a"
-					(reference "#PWR037")
+					(reference "#PWR050")
 					(unit 1)
 				)
@@
 		(in_pos_files yes)
 		(dnp no)
-		(property "Reference" "#PWR045"
+		(property "Reference" "#PWR057"
 			(at 218.44 100.33 0)
 			(hide yes)
@@
 			(project "stm32f103c8t6"
 				(path "/bd823326-686b-4669-b4e8-652a43eb6bb4/b6e9bfc2-4cf7-4d7e-81c9-9912399d557a"
-					(reference "#PWR045")
+					(reference "#PWR057")
 					(unit 1)
 				)
@@
 		(dnp no)
 		(fields_autoplaced yes)
-		(property "Reference" "U3"
+		(property "Reference" "U4"
 			(at 160.8933 67.31 0)
 			(show_name no)
@@
 			(project "stm32f103c8t6"
 				(path "/bd823326-686b-4669-b4e8-652a43eb6bb4/b6e9bfc2-4cf7-4d7e-81c9-9912399d557a"
-					(reference "U3")
+					(reference "U4")
 					(unit 1)
 				)
@@
 		(dnp no)
 		(fields_autoplaced yes)
-		(property "Reference" "C17"
+		(property "Reference" "C19"
 			(at 182.88 44.4499 0)
 			(show_name no)
@@
 			(project "stm32f103c8t6"
 				(path "/bd823326-686b-4669-b4e8-652a43eb6bb4/b6e9bfc2-4cf7-4d7e-81c9-9912399d557a"
-					(reference "C17")
+					(reference "C19")
 					(unit 1)
 				)
@@
 			)
 		)
-		(property "Footprint" ""
+		(property "Footprint" "LED_SMD:LED_0603_1608Metric"
 			(at 187.96 101.6 0)
 			(hide yes)
@@
 			)
 		)
-		(property "Footprint" ""
+		(property "Footprint" "LED_SMD:LED_0603_1608Metric"
 			(at 187.96 104.14 0)
 			(hide yes)
@@
 				(path "/bd823326-686b-4669-b4e8-652a43eb6bb4/b6e9bfc2-4cf7-4d7e-81c9-9912399d557a"
 					(reference "D6")
+					(unit 1)
+				)
+			)
+		)
+	)
+	(symbol
+		(lib_id "power:GND")
+		(at 132.08 118.11 0)
+		(unit 1)
+		(body_style 1)
+		(exclude_from_sim no)
+		(in_bom yes)
+		(on_board yes)
+		(in_pos_files yes)
+		(dnp no)
+		(fields_autoplaced yes)
+		(property "Reference" "#PWR058"
+			(at 132.08 124.46 0)
+			(hide yes)
+			(show_name no)
+			(do_not_autoplace no)
+			(effects
+				(font
+					(size 1.27 1.27)
+				)
+			)
+		)
+		(property "Value" "GND"
+			(at 132.08 123.19 0)
+			(show_name no)
+			(do_not_autoplace no)
+			(effects
+				(font
+					(size 1.27 1.27)
+				)
+			)
+		)
+		(property "Footprint" ""
+			(at 132.08 118.11 0)
+			(hide yes)
+			(show_name no)
+			(do_not_autoplace no)
+			(effects
+				(font
+					(size 1.27 1.27)
+				)
+			)
+		)
+		(property "Datasheet" ""
+			(at 132.08 118.11 0)
+			(hide yes)
+			(show_name no)
+			(do_not_autoplace no)
+			(effects
+				(font
+					(size 1.27 1.27)
+				)
+			)
+		)
+		(property "Description" "Power symbol creates a global label with name \"GND\" , ground"
+			(at 132.08 118.11 0)
+			(hide yes)
+			(show_name no)
+			(do_not_autoplace no)
+			(effects
+				(font
+					(size 1.27 1.27)
+				)
+			)
+		)
+		(pin "1"
+		)
+		(instances
+			(project "stm32f103c8t6"
+				(path "/bd823326-686b-4669-b4e8-652a43eb6bb4/b6e9bfc2-4cf7-4d7e-81c9-9912399d557a"
+					(reference "#PWR058")
 					(unit 1)
 				)
@@
 		(dnp no)
 		(fields_autoplaced yes)
-		(property "Reference" "#PWR042"
+		(property "Reference" "#PWR056"
 			(at 207.01 74.93 0)
 			(hide yes)
@@
 			(project "stm32f103c8t6"
 				(path "/bd823326-686b-4669-b4e8-652a43eb6bb4/b6e9bfc2-4cf7-4d7e-81c9-9912399d557a"
-					(reference "#PWR042")
+					(reference "#PWR056")
 					(unit 1)
 				)
@@
 		(in_pos_files yes)
 		(dnp no)
-		(property "Reference" "#PWR038"
+		(property "Reference" "#PWR049"
 			(at 114.3 36.83 0)
 			(hide yes)
@@
 			(project "stm32f103c8t6"
 				(path "/bd823326-686b-4669-b4e8-652a43eb6bb4/b6e9bfc2-4cf7-4d7e-81c9-9912399d557a"
-					(reference "#PWR038")
+					(reference "#PWR049")
 					(unit 1)
 				)
@@
 		(in_pos_files yes)
 		(dnp no)
-		(property "Reference" "#PWR041"
+		(property "Reference" "#PWR055"
 			(at 179.07 30.48 0)
 			(hide yes)
@@
 			(project "stm32f103c8t6"
 				(path "/bd823326-686b-4669-b4e8-652a43eb6bb4/b6e9bfc2-4cf7-4d7e-81c9-9912399d557a"
-					(reference "#PWR041")
+					(reference "#PWR055")
 					(unit 1)
 				)
@@
 		(in_pos_files yes)
 		(dnp no)
-		(property "Reference" "R23"
+		(property "Reference" "R34"
 			(at 205.74 106.68 90)
 			(show_name no)
@@
 			)
 		)
-		(property "Footprint" ""
+		(property "Footprint" "Resistor_SMD:R_0603_1608Metric"
 			(at 205.994 105.156 90)
 			(hide yes)
@@
 			(project "stm32f103c8t6"
 				(path "/bd823326-686b-4669-b4e8-652a43eb6bb4/b6e9bfc2-4cf7-4d7e-81c9-9912399d557a"
-					(reference "R23")
+					(reference "R34")
 					(unit 1)
 				)
@@
 		(dnp no)
 		(fields_autoplaced yes)
-		(property "Reference" "C16"
+		(property "Reference" "C17"
 			(at 118.11 44.4499 0)
 			(show_name no)
@@
 			(project "stm32f103c8t6"
 				(path "/bd823326-686b-4669-b4e8-652a43eb6bb4/b6e9bfc2-4cf7-4d7e-81c9-9912399d557a"
-					(reference "C16")
+					(reference "C17")
 					(unit 1)
 				)
@@
 		(in_pos_files yes)
 		(dnp no)
-		(property "Reference" "R21"
+		(property "Reference" "R32"
 			(at 117.856 92.964 90)
 			(show_name no)
@@
 			)
 		)
-		(property "Footprint" ""
+		(property "Footprint" "Resistor_SMD:R_0603_1608Metric"
 			(at 121.666 94.996 90)
 			(hide yes)
@@
 			(project "stm32f103c8t6"
 				(path "/bd823326-686b-4669-b4e8-652a43eb6bb4/b6e9bfc2-4cf7-4d7e-81c9-9912399d557a"
-					(reference "R21")
+					(reference "R32")
 					(unit 1)
 				)
@@
 		(in_pos_files yes)
 		(dnp no)
-		(property "Reference" "#PWR035"
+		(property "Reference" "#PWR052"
 			(at 153.67 64.77 0)
 			(hide yes)
@@
 			(project "stm32f103c8t6"
 				(path "/bd823326-686b-4669-b4e8-652a43eb6bb4/b6e9bfc2-4cf7-4d7e-81c9-9912399d557a"
-					(reference "#PWR035")
+					(reference "#PWR052")
 					(unit 1)
 				)
@@
 		(dnp no)
 		(fields_autoplaced yes)
-		(property "Reference" "C18"
+		(property "Reference" "C20"
 			(at 210.82 44.4499 0)
 			(show_name no)
@@
 			(project "stm32f103c8t6"
 				(path "/bd823326-686b-4669-b4e8-652a43eb6bb4/b6e9bfc2-4cf7-4d7e-81c9-9912399d557a"
-					(reference "C18")
+					(reference "C20")
 					(unit 1)
 				)
@@
 		(dnp no)
 		(fields_autoplaced yes)
-		(property "Reference" "#PWR043"
+		(property "Reference" "#PWR048"
 			(at 101.6 76.2 0)
 			(hide yes)
@@
 			(project "stm32f103c8t6"
 				(path "/bd823326-686b-4669-b4e8-652a43eb6bb4/b6e9bfc2-4cf7-4d7e-81c9-9912399d557a"
-					(reference "#PWR043")
+					(reference "#PWR048")
 					(unit 1)
 				)
@@
 		(in_pos_files yes)
 		(dnp no)
-		(property "Reference" "#PWR044"
+		(property "Reference" "#PWR047"
 			(at 110.49 93.98 0)
 			(hide yes)
@@
 			(project "stm32f103c8t6"
 				(path "/bd823326-686b-4669-b4e8-652a43eb6bb4/b6e9bfc2-4cf7-4d7e-81c9-9912399d557a"
-					(reference "#PWR044")
+					(reference "#PWR047")
 					(unit 1)
 				)
