File: led.kicad_sch (KiCad schematic)
At the start: 8 parts

Commit message: Update USB-C and FTDI circuits and add button and potentiometer sheets
Parts:
- D1: value LED -> LED(RED)
- D2: value LED -> LED(GREEN)
- D3: value LED -> LED(BLUE)
- D4: value LED -> LED(ORANGE)
- R2, R5: value 10KR(1608) -> 270R(1608)
- R3, R4: value 10KR(1608) -> 62R(1608)

Commit message: Update schematics, power flags and PCB design
Parts:
- D1, D2, D3, D4: footprint (none) -> LED_SMD:LED_0603_1608Metric
- R16: renamed from R2; footprint (none) -> Resistor_SMD:R_0603_1608Metric
- R17: renamed from R3; footprint (none) -> Resistor_SMD:R_0603_1608Metric
- R18: renamed from R4; footprint (none) -> Resistor_SMD:R_0603_1608Metric
- R19: renamed from R5; footprint (none) -> Resistor_SMD:R_0603_1608Metric
Changed lines of the file:
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@@
 		(in_pos_files yes)
 		(dnp no)
-		(property "Reference" "R5"
+		(property "Reference" "R19"
 			(at 53.34 87.63 90)
 			(show_name no)
@@
 			)
 		)
-		(property "Footprint" ""
+		(property "Footprint" "Resistor_SMD:R_0603_1608Metric"
 			(at 53.594 89.154 90)
 			(hide yes)
@@
 			(project "stm32f103c8t6"
 				(path "/bd823326-686b-4669-b4e8-652a43eb6bb4/417559c3-f209-435e-9a7f-a3295fb9237d"
-					(reference "R5")
+					(reference "R19")
 					(unit 1)
 				)
@@
 			)
 		)
-		(property "Footprint" ""
+		(property "Footprint" "LED_SMD:LED_0603_1608Metric"
 			(at 71.12 64.77 0)
 			(hide yes)
@@
 			)
 		)
-		(property "Footprint" ""
+		(property "Footprint" "LED_SMD:LED_0603_1608Metric"
 			(at 71.12 49.53 0)
 			(hide yes)
@@
 			)
 		)
-		(property "Footprint" ""
+		(property "Footprint" "LED_SMD:LED_0603_1608Metric"
 			(at 71.12 90.17 0)
 			(hide yes)
@@
 		(dnp no)
 		(fields_autoplaced yes)
-		(property "Reference" "#PWR017"
+		(property "Reference" "#PWR030"
 			(at 33.02 48.26 0)
 			(hide yes)
@@
 			(project "stm32f103c8t6"
 				(path "/bd823326-686b-4669-b4e8-652a43eb6bb4/417559c3-f209-435e-9a7f-a3295fb9237d"
-					(reference "#PWR017")
+					(reference "#PWR030")
 					(unit 1)
 				)
@@
 		(in_pos_files yes)
 		(dnp no)
-		(property "Reference" "R2"
+		(property "Reference" "R16"
 			(at 53.34 46.99 90)
 			(show_name no)
@@
 			)
 		)
-		(property "Footprint" ""
+		(property "Footprint" "Resistor_SMD:R_0603_1608Metric"
 			(at 53.594 48.514 90)
 			(hide yes)
@@
 			(project "stm32f103c8t6"
 				(path "/bd823326-686b-4669-b4e8-652a43eb6bb4/417559c3-f209-435e-9a7f-a3295fb9237d"
-					(reference "R2")
+					(reference "R16")
 					(unit 1)
 				)
@@
 			)
 		)
-		(property "Footprint" ""
+		(property "Footprint" "LED_SMD:LED_0603_1608Metric"
 			(at 71.12 77.47 0)
 			(hide yes)
@@
 		(in_pos_files yes)
 		(dnp no)
-		(property "Reference" "R4"
+		(property "Reference" "R18"
 			(at 53.34 74.93 90)
 			(show_name no)
@@
 			)
 		)
-		(property "Footprint" ""
+		(property "Footprint" "Resistor_SMD:R_0603_1608Metric"
 			(at 53.594 76.454 90)
 			(hide yes)
@@
 			(project "stm32f103c8t6"
 				(path "/bd823326-686b-4669-b4e8-652a43eb6bb4/417559c3-f209-435e-9a7f-a3295fb9237d"
-					(reference "R4")
+					(reference "R18")
 					(unit 1)
 				)
@@
 		(in_pos_files yes)
 		(dnp no)
-		(property "Reference" "R3"
+		(property "Reference" "R17"
 			(at 53.34 62.23 90)
 			(show_name no)
@@
 			)
 		)
-		(property "Footprint" ""
+		(property "Footprint" "Resistor_SMD:R_0603_1608Metric"
 			(at 53.594 63.754 90)
 			(hide yes)
@@
 			(project "stm32f103c8t6"
 				(path "/bd823326-686b-4669-b4e8-652a43eb6bb4/417559c3-f209-435e-9a7f-a3295fb9237d"
-					(reference "R3")
-					(unit 1)
-				)
+					(reference "R17")
+					(unit 1)
+				)
