File: pot.kicad_sch (KiCad schematic)
At the start: 12 parts

Commit message: Update schematics, power flags and PCB design
Parts:
- R28: renamed from R15; footprint (none) -> Resistor_SMD:R_0603_1608Metric
- R29: renamed from R16; footprint (none) -> Resistor_SMD:R_0603_1608Metric
- R30: renamed from R17; footprint (none) -> Resistor_SMD:R_0603_1608Metric
- R31: renamed from R18; footprint (none) -> Resistor_SMD:R_0603_1608Metric
- RV1, RV2, RV3, RV4: footprint Package_SO:TSSOP-20_4.4x6.5mm_P0.65mm -> Potentiometer_THT:Potentiometer_Alps_RK09K_Single_Vertical
- renumbered C12 to C13, C13 to C14, C14 to C15, C15 to C16
Changed lines of the file:
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@@
 			)
 		)
-		(property "Footprint" "Package_SO:TSSOP-20_4.4x6.5mm_P0.65mm"
+		(property "Footprint" "Potentiometer_THT:Potentiometer_Alps_RK09K_Single_Vertical"
 			(at 97.79 82.55 0)
 			(hide yes)
@@
 		(dnp no)
 		(fields_autoplaced yes)
-		(property "Reference" "#PWR032"
+		(property "Reference" "#PWR044"
 			(at 161.29 116.84 0)
 			(hide yes)
@@
 			(project "stm32f103c8t6"
 				(path "/bd823326-686b-4669-b4e8-652a43eb6bb4/44ab54ba-53a5-410a-906a-77df5de9df15"
-					(reference "#PWR032")
+					(reference "#PWR044")
 					(unit 1)
 				)
@@
 		(dnp no)
 		(fields_autoplaced yes)
-		(property "Reference" "C12"
+		(property "Reference" "C13"
 			(at 54.61 86.3599 0)
 			(show_name no)
@@
 			(project "stm32f103c8t6"
 				(path "/bd823326-686b-4669-b4e8-652a43eb6bb4/44ab54ba-53a5-410a-906a-77df5de9df15"
-					(reference "C12")
+					(reference "C13")
 					(unit 1)
 				)
@@
 		(dnp no)
 		(fields_autoplaced yes)
-		(property "Reference" "R17"
+		(property "Reference" "R30"
 			(at 172.72 77.47 90)
 			(show_name no)
@@
 			)
 		)
-		(property "Footprint" ""
+		(property "Footprint" "Resistor_SMD:R_0603_1608Metric"
 			(at 172.974 82.804 90)
 			(hide yes)
@@
 			(project "stm32f103c8t6"
 				(path "/bd823326-686b-4669-b4e8-652a43eb6bb4/44ab54ba-53a5-410a-906a-77df5de9df15"
-					(reference "R17")
+					(reference "R30")
 					(unit 1)
 				)
@@
 			)
 		)
-		(property "Footprint" "Package_SO:TSSOP-20_4.4x6.5mm_P0.65mm"
+		(property "Footprint" "Potentiometer_THT:Potentiometer_Alps_RK09K_Single_Vertical"
 			(at 161.29 83.82 0)
 			(hide yes)
@@
 		(dnp no)
 		(fields_autoplaced yes)
-		(property "Reference" "#PWR028"
+		(property "Reference" "#PWR040"
 			(at 27.94 115.57 0)
 			(hide yes)
@@
 			(project "stm32f103c8t6"
 				(path "/bd823326-686b-4669-b4e8-652a43eb6bb4/44ab54ba-53a5-410a-906a-77df5de9df15"
-					(reference "#PWR028")
+					(reference "#PWR040")
 					(unit 1)
 				)
@@
 		(dnp no)
 		(fields_autoplaced yes)
-		(property "Reference" "C15"
+		(property "Reference" "C16"
 			(at 251.46 87.6299 0)
 			(show_name no)
@@
 			(project "stm32f103c8t6"
 				(path "/bd823326-686b-4669-b4e8-652a43eb6bb4/44ab54ba-53a5-410a-906a-77df5de9df15"
-					(reference "C15")
+					(reference "C16")
 					(unit 1)
 				)
@@
 		(dnp no)
 		(fields_autoplaced yes)
-		(property "Reference" "#PWR034"
+		(property "Reference" "#PWR046"
 			(at 224.79 116.84 0)
 			(hide yes)
@@
 			(project "stm32f103c8t6"
 				(path "/bd823326-686b-4669-b4e8-652a43eb6bb4/44ab54ba-53a5-410a-906a-77df5de9df15"
-					(reference "#PWR034")
+					(reference "#PWR046")
 					(unit 1)
 				)
@@
 		(dnp no)
 		(fields_autoplaced yes)
-		(property "Reference" "#PWR027"
+		(property "Reference" "#PWR039"
 			(at 27.94 73.66 0)
 			(hide yes)
@@
 			(project "stm32f103c8t6"
 				(path "/bd823326-686b-4669-b4e8-652a43eb6bb4/44ab54ba-53a5-410a-906a-77df5de9df15"
-					(reference "#PWR027")
+					(reference "#PWR039")
 					(unit 1)
 				)
@@
 		(dnp no)
 		(fields_autoplaced yes)
-		(property "Reference" "R15"
+		(property "Reference" "R28"
 			(at 39.37 76.2 90)
 			(show_name no)
@@
 			)
 		)
-		(property "Footprint" ""
+		(property "Footprint" "Resistor_SMD:R_0603_1608Metric"
 			(at 39.624 81.534 90)
 			(hide yes)
@@
 			(project "stm32f103c8t6"
 				(path "/bd823326-686b-4669-b4e8-652a43eb6bb4/44ab54ba-53a5-410a-906a-77df5de9df15"
-					(reference "R15")
+					(reference "R28")
 					(unit 1)
 				)
@@
 		(dnp no)
 		(fields_autoplaced yes)
-		(property "Reference" "R16"
+		(property "Reference" "R29"
 			(at 109.22 76.2 90)
 			(show_name no)
@@
 			)
 		)
-		(property "Footprint" ""
+		(property "Footprint" "Resistor_SMD:R_0603_1608Metric"
 			(at 109.474 81.534 90)
 			(hide yes)
@@
 			(project "stm32f103c8t6"
 				(path "/bd823326-686b-4669-b4e8-652a43eb6bb4/44ab54ba-53a5-410a-906a-77df5de9df15"
-					(reference "R16")
+					(reference "R29")
 					(unit 1)
 				)
@@
 		(dnp no)
 		(fields_autoplaced yes)
-		(property "Reference" "C14"
+		(property "Reference" "C15"
 			(at 187.96 87.6299 0)
 			(show_name no)
@@
 			(project "stm32f103c8t6"
 				(path "/bd823326-686b-4669-b4e8-652a43eb6bb4/44ab54ba-53a5-410a-906a-77df5de9df15"
-					(reference "C14")
+					(reference "C15")
 					(unit 1)
 				)
@@
 		(dnp no)
 		(fields_autoplaced yes)
-		(property "Reference" "#PWR030"
+		(property "Reference" "#PWR042"
 			(at 97.79 115.57 0)
 			(hide yes)
@@
 			(project "stm32f103c8t6"
 				(path "/bd823326-686b-4669-b4e8-652a43eb6bb4/44ab54ba-53a5-410a-906a-77df5de9df15"
-					(reference "#PWR030")
+					(reference "#PWR042")
 					(unit 1)
 				)
@@
 		(dnp no)
 		(fields_autoplaced yes)
-		(property "Reference" "#PWR033"
+		(property "Reference" "#PWR045"
 			(at 224.79 74.93 0)
 			(hide yes)
@@
 			(project "stm32f103c8t6"
 				(path "/bd823326-686b-4669-b4e8-652a43eb6bb4/44ab54ba-53a5-410a-906a-77df5de9df15"
-					(reference "#PWR033")
+					(reference "#PWR045")
 					(unit 1)
 				)
@@
 			)
 		)
-		(property "Footprint" "Package_SO:TSSOP-20_4.4x6.5mm_P0.65mm"
+		(property "Footprint" "Potentiometer_THT:Potentiometer_Alps_RK09K_Single_Vertical"
 			(at 27.94 82.55 0)
 			(hide yes)
@@
 		(dnp no)
 		(fields_autoplaced yes)
-		(property "Reference" "C13"
+		(property "Reference" "C14"
 			(at 124.46 86.3599 0)
 			(show_name no)
@@
 			(project "stm32f103c8t6"
 				(path "/bd823326-686b-4669-b4e8-652a43eb6bb4/44ab54ba-53a5-410a-906a-77df5de9df15"
-					(reference "C13")
+					(reference "C14")
 					(unit 1)
 				)
@@
 		(dnp no)
 		(fields_autoplaced yes)
-		(property "Reference" "#PWR029"
+		(property "Reference" "#PWR041"
 			(at 97.79 73.66 0)
 			(hide yes)
@@
 			(project "stm32f103c8t6"
 				(path "/bd823326-686b-4669-b4e8-652a43eb6bb4/44ab54ba-53a5-410a-906a-77df5de9df15"
-					(reference "#PWR029")
+					(reference "#PWR041")
 					(unit 1)
 				)
@@
 		(dnp no)
 		(fields_autoplaced yes)
-		(property "Reference" "#PWR031"
+		(property "Reference" "#PWR043"
 			(at 161.29 74.93 0)
 			(hide yes)
@@
 			(project "stm32f103c8t6"
 				(path "/bd823326-686b-4669-b4e8-652a43eb6bb4/44ab54ba-53a5-410a-906a-77df5de9df15"
-					(reference "#PWR031")
+					(reference "#PWR043")
 					(unit 1)
 				)
@@
 		(dnp no)
 		(fields_autoplaced yes)
-		(property "Reference" "R18"
+		(property "Reference" "R31"
 			(at 236.22 77.47 90)
 			(show_name no)
@@
 			)
 		)
-		(property "Footprint" ""
+		(property "Footprint" "Resistor_SMD:R_0603_1608Metric"
 			(at 236.474 82.804 90)
 			(hide yes)
@@
 			(project "stm32f103c8t6"
 				(path "/bd823326-686b-4669-b4e8-652a43eb6bb4/44ab54ba-53a5-410a-906a-77df5de9df15"
-					(reference "R18")
+					(reference "R31")
 					(unit 1)
 				)
@@
 			)
 		)
-		(property "Footprint" "Package_SO:TSSOP-20_4.4x6.5mm_P0.65mm"
+		(property "Footprint" "Potentiometer_THT:Potentiometer_Alps_RK09K_Single_Vertical"
 			(at 224.79 83.82 0)
 			(hide yes)
